Commit message: update

File: src/urdfs/urdf/camera.xacro (robot description, xacro)
@@ -22,5 +22,5 @@
         <parent link="base_link" />
         <child link="camera_link" />
-        <origin xyz="${(0.4 + camera_length) / 2.0} 0 ${0.1 / 2.0}" rpy="0 0 0" />
+        <origin xyz="${(0.6 + camera_length) / 2.0} 0 ${0.25 / 2.0}" rpy="0 0 0" />
     </joint>
     <link name="camera_link_optical" />

File: src/urdfs/urdf/gazebo_plugin.xacro (robot description, xacro)
@@ -1,16 +1,14 @@
 <?xml version="1.0"?>
 <robot xmlns:xacro="http://www.ros.org/wiki/xacro">
-    <gazebo reference="caster_wheel">
-        <mu1 value="0.01" />
-        <mu2 value="0.01" />
-    </gazebo>
     <gazebo>
         <plugin
             filename="gz-sim-diff-drive-system"
             name="gz::sim::systems::DiffDrive">
-            <left_joint>base_left_wheel_joint</left_joint>
-            <right_joint>base_right_wheel_joint</right_joint>
-            <wheel_separation>0.23</wheel_separation>
-            <wheel_radius>0.05</wheel_radius>
+            <left_joint>base_frontleft_wheel_joint</left_joint>
+            <left_joint>base_rearleft_wheel_joint</left_joint>
+            <right_joint>base_frontright_wheel_joint</right_joint>
+            <right_joint>base_rearright_wheel_joint</right_joint>
+            <wheel_separation>0.5</wheel_separation>
+            <wheel_radius>0.1</wheel_radius>
             <frame_id>odom</frame_id>
             <child_frame_id>zippy</child_frame_id>
@@ -21,6 +19,8 @@
             filename="gz-sim-joint-state-publisher-system"
             name="gz::sim::systems::JointStatePublisher">
-            <joint_name>base_left_wheel_joint</joint_name>
-            <joint_name>base_right_wheel_joint</joint_name>
+            <joint_name>base_frontleft_wheel_joint</joint_name>
+            <joint_name>base_frontright_wheel_joint</joint_name>
+            <joint_name>base_rearleft_wheel_joint</joint_name>
+            <joint_name>base_rearright_wheel_joint</joint_name>
         </plugin>
     </gazebo>

File: src/urdfs/urdf/imu_sensor.xacro (robot description, xacro)
@@ -23,5 +23,5 @@
         <parent link="base_link" />
         <child link="imu_link" />
-        <origin xyz="0 0 ${0.1 + (imu_height)}" rpy="0 0 0" />
+        <origin xyz="0 0 ${0.25 + (imu_height)}" rpy="0 0 0" />
     </joint>
     <gazebo reference="imu_link">

File: src/urdfs/urdf/lidar.xacro (robot description, xacro)
@@ -22,5 +22,5 @@
         <parent link="base_link" />
         <child link="lidar_link" />
-        <origin xyz="0 0 ${0.1 + (lidar_height) / 2.0}" rpy="0 0 0" />
+        <origin xyz="0 0 ${0.25 + (lidar_height) / 2.0}" rpy="0 0 0" />
     </joint>
     <link name="lidar_link_optical"/>

File: src/urdfs/urdf/ros2_hardwareinterface.xacro (robot description, xacro)
@@ -5,10 +5,20 @@
             <plugin>gz_ros2_control/GazeboSimSystem</plugin>
         </hardware>
-        <joint name="base_right_wheel_joint">
+        <joint name="base_frontleft_wheel_joint">
             <command_interface name="velocity"/>
             <state_interface name="velocity"/>
             <state_interface name="position"/>
         </joint>
-        <joint name="base_left_wheel_joint">
+        <joint name="base_frontright_wheel_joint">
+            <command_interface name="velocity"/>
+            <state_interface name="velocity"/>
+            <state_interface name="position"/>
+        </joint>
+        <joint name="base_rearleft_wheel_joint">
+            <command_interface name="velocity"/>
+            <state_interface name="velocity"/>
+            <state_interface name="position"/>
+        </joint>
+        <joint name="base_rearright_wheel_joint">
             <command_interface name="velocity"/>
             <state_interface name="velocity"/>

File: src/urdfs/urdf/zippy.urdf.xacro (robot description, xacro)
@@ -9,8 +9,16 @@
     <xacro:include filename="gazebo_plugin.xacro" />
     <xacro:include filename="ros2_hardwareinterface.xacro" />
-    <xacro:property name="zippy_radius" value="0.2" />
-    <xacro:property name="zippy_height" value="0.1" />
-    <xacro:property name="wheel_radius" value="0.05" />
-    <xacro:property name="wheel_thickness" value="0.03" />
+    <xacro:property name="chassis_length" value="0.6" />
+    <xacro:property name="chassis_width" value="0.45" />
+    <xacro:property name="chassis_height" value="0.25" />
+    <xacro:property name="chassis_mass" value="25.0" />
+    <xacro:property name="wheel_radius" value="0.1" />
+    <xacro:property name="wheel_thickness" value="0.06" />
+    <xacro:property name="wheel_mass" value="1.5" />
+    <!-- Distance between left/right wheel centers and front/rear wheel centers -->
+    <xacro:property name="track_width" value="0.5" />
+    <xacro:property name="wheelbase" value="0.45" />
+    <!-- Height of the chassis center above the ground (wheel axle height) -->
+    <xacro:property name="chassis_z" value="${wheel_radius}" />
     <link name="zippy">
     </link>
@@ -18,16 +26,16 @@
         <visual>
             <geometry>
-                <cylinder radius="${zippy_radius}" length="${zippy_height}" />
+                <box size="${chassis_length} ${chassis_width} ${chassis_height}" />
             </geometry>
-            <origin xyz="0 0 ${wheel_radius}" rpy="0 0 0" />
+            <origin xyz="0 0 ${chassis_z}" rpy="0 0 0" />
             <material name="blue" />
         </visual>
         <collision>
             <geometry>
-                <cylinder radius="${zippy_radius}" length="${zippy_height}" />
+                <box size="${chassis_length} ${chassis_width} ${chassis_height}" />
             </geometry>
-            <origin xyz="0 0 ${wheel_radius}" rpy="0 0 0" />
+            <origin xyz="0 0 ${chassis_z}" rpy="0 0 0" />
         </collision>
-        <xacro:cylinder_inertia Mass="10.0" r="${zippy_radius}" h="${zippy_height}" arr_xyz="0 0 ${wheel_radius}" arr_rpy="0 0 0" />
+        <xacro:box_inertia Mass="${chassis_mass}" x="${chassis_length}" y="${chassis_width}" z="${chassis_height}" arr_xyz="0 0 ${chassis_z}" arr_rpy="0 0 0" />
     </link>
     <xacro:macro name="wheel" params="params">
@@ -46,70 +54,60 @@
                 <origin xyz="0 0 0" rpy="${pi/2} 0 0"/>
             </collision>
-            <xacro:cylinder_inertia Mass="1.0" r="${wheel_radius}" h="${wheel_thickness}" arr_xyz="0 0 0" arr_rpy="${pi/2} 0 0"/>
+            <xacro:cylinder_inertia Mass="${wheel_mass}" r="${wheel_radius}" h="${wheel_thickness}" arr_xyz="0 0 0" arr_rpy="${pi/2} 0 0"/>
         </link>
     </xacro:macro>
-    <xacro:wheel params="right_wheel" />
-    <xacro:wheel params="left_wheel" />
-    <link name="caster_wheel">
-        <visual>
-            <geometry>
-                <sphere radius="0.025"/>
-            </geometry>
-            <origin xyz="0 0 0" rpy="0 0 0"/>
-            <material name="grey"/>
-        </visual>
-        <collision>
-            <geometry>
-                <sphere radius="0.025"/>
-            </geometry>
-            <origin xyz="0 0 0" rpy="0 0 0"/>
-        </collision>
-        <xacro:solid_sphere_inertia Mass="0.5" r="0.025" arr_xyz="0 0 0" arr_rpy="0 0 0"/>
-    </link>
-    <joint name="base_right_wheel_joint" type="continuous">
+    <xacro:wheel params="front_left_wheel" />
+    <xacro:wheel params="front_right_wheel" />
+    <xacro:wheel params="rear_left_wheel" />
+    <xacro:wheel params="rear_right_wheel" />
+    <joint name="base_frontleft_wheel_joint" type="continuous">
         <parent link="base_link"/>
-        <child link="right_wheel"/>
-        <origin xyz="${-zippy_radius/2} ${-zippy_radius/2 - wheel_thickness/2} 0" rpy="0 0 0"/>
+        <child link="front_left_wheel"/>
+        <origin xyz="${wheelbase/2} ${track_width/2} 0" rpy="0 0 0"/>
         <axis xyz="0 1 0"/>
     </joint>
-    <joint name="base_left_wheel_joint" type="continuous">
+    <joint name="base_frontright_wheel_joint" type="continuous">
         <parent link="base_link"/>
-        <child link="left_wheel"/>
-        <origin xyz="${-zippy_radius/2} ${zippy_radius/2 + wheel_thickness/2} 0" rpy="0 0 0"/>
+        <child link="front_right_wheel"/>
+        <origin xyz="${wheelbase/2} ${-track_width/2} 0" rpy="0 0 0"/>
         <axis xyz="0 1 0"/>
     </joint>
-    <joint name="base_caster_wheel_joint" type="fixed">
+    <joint name="base_rearleft_wheel_joint" type="continuous">
         <parent link="base_link"/>
-        <child link="caster_wheel"/>
-        <origin xyz="${zippy_radius/4} 0 ${-wheel_radius/2}" rpy="0 0 0"/>
+        <child link="rear_left_wheel"/>
+        <origin xyz="${-wheelbase/2} ${track_width/2} 0" rpy="0 0 0"/>
+        <axis xyz="0 1 0"/>
+    </joint>
+    <joint name="base_rearright_wheel_joint" type="continuous">
+        <parent link="base_link"/>
+        <child link="rear_right_wheel"/>
+        <origin xyz="${-wheelbase/2} ${-track_width/2} 0" rpy="0 0 0"/>
+        <axis xyz="0 1 0"/>
     </joint>
     <joint name="spine" type="fixed">
         <parent link="zippy"/>
         <child link="base_link"/>
-        <origin xyz="0 0 ${wheel_radius}" rpy="0 0 0"/>
+        <origin xyz="0 0 ${chassis_z}" rpy="0 0 0"/>
     </joint>
-    <gazebo reference="caster_wheel">
-        <mu1 value="0.01" />
-        <mu2 value="0.01" />
-    </gazebo>
-        <!-- Wheels -->
-    <gazebo reference="left_wheel">
-        <mu1>1000000000000000.0</mu1>
-        <mu2>1000000000000000.0</mu2>
-        <kp>1000000000000.0</kp>
-        <kd>10.0</kd>
-        <minDepth>0.001</minDepth>
-        <maxVel>0.1</maxVel>
-        <fdir1>1 0 0</fdir1>
-    </gazebo>
-    <gazebo reference="right_wheel">
-        <mu1>1000000000000000.0</mu1>
-        <mu2>1000000000000000.0</mu2>
-        <kp>1000000000000.0</kp>
-        <kd>10.0</kd>
-        <minDepth>0.001</minDepth>
-        <maxVel>0.1</maxVel>
-        <fdir1>1 0 0</fdir1>
-    </gazebo>
+    <!-- Wheels: high longitudinal (rolling-direction) friction, matching the
+         original tuning. Skid-steer relies on lateral wheel scrub to turn,
+         so mu2 could be tuned lower than mu1 for more realistic slip - left
+         as-is here to match the previous friction tuning; revisit if the
+         sim turning behavior looks wrong. -->
+    <xacro:macro name="wheel_friction" params="link">
+        <gazebo reference="${link}">
+            <mu1>1000000000000000.0</mu1>
+            <mu2>1000000000000000.0</mu2>
+            <kp>1000000000000.0</kp>
+            <kd>10.0</kd>
+            <minDepth>0.001</minDepth>
+            <maxVel>0.1</maxVel>
+            <fdir1>1 0 0</fdir1>
+        </gazebo>
+    </xacro:macro>
+    <xacro:wheel_friction link="front_left_wheel" />
+    <xacro:wheel_friction link="front_right_wheel" />
+    <xacro:wheel_friction link="rear_left_wheel" />
+    <xacro:wheel_friction link="rear_right_wheel" />
     <gazebo>
         <plugin filename="gz_ros2_control-system" name="gz_ros2_control::GazeboSimROS2ControlPlugin">
