Commit message: update

File: src/urdfs/urdf/zippy.urdf.xacro (robot description, xacro)
@@ -90,10 +90,5 @@
         <origin xyz="0 0 ${chassis_z}" rpy="0 0 0"/>
     </joint>
-    <!-- Wheels: high longitudinal (rolling-direction) friction, matching the
-         original tuning. Skid-steer relies on lateral wheel scrub to turn,
-         so mu2 could be tuned lower than mu1 for more realistic slip - left
-         as-is here to match the previous friction tuning; revisit if the
-         sim turning behavior looks wrong. -->
-    <xacro:macro name="wheel_friction" params="link">
+    <!-- <xacro:macro name="wheel_friction" params="link">
         <gazebo reference="${link}">
             <mu1>1000000000000000.0</mu1>
@@ -109,5 +104,5 @@
     <xacro:wheel_friction link="front_right_wheel" />
     <xacro:wheel_friction link="rear_left_wheel" />
-    <xacro:wheel_friction link="rear_right_wheel" />
+    <xacro:wheel_friction link="rear_right_wheel" /> -->
     <gazebo>
         <plugin filename="gz_ros2_control-system" name="gz_ros2_control::GazeboSimROS2ControlPlugin">
@@ -115,9 +110,9 @@
         </plugin>
     </gazebo>
-    <gazebo>
+    <!-- <gazebo>
         <plugin name='gz::sim::systems::Sensors' filename='gz-sim-sensors-system'>
         <render_engine>ogre2</render_engine>
         </plugin>
         <plugin name='gz::sim::systems::Imu' filename='gz-sim-imu-system'/>
-    </gazebo>
+    </gazebo> -->
 </robot>

Commit message: update

File: src/urdfs/urdf/zippy.urdf.xacro (robot description, xacro)
@@ -90,5 +90,5 @@
         <origin xyz="0 0 ${chassis_z}" rpy="0 0 0"/>
     </joint>
-    <!-- <xacro:macro name="wheel_friction" params="link">
+    <xacro:macro name="wheel_friction" params="link">
         <gazebo reference="${link}">
             <mu1>1000000000000000.0</mu1>
@@ -104,5 +104,5 @@
     <xacro:wheel_friction link="front_right_wheel" />
     <xacro:wheel_friction link="rear_left_wheel" />
-    <xacro:wheel_friction link="rear_right_wheel" /> -->
+    <xacro:wheel_friction link="rear_right_wheel" />
     <gazebo>
         <plugin filename="gz_ros2_control-system" name="gz_ros2_control::GazeboSimROS2ControlPlugin">

Commit message: update

File: src/urdfs/urdf/zippy.urdf.xacro (robot description, xacro)
@@ -12,8 +12,8 @@
     <xacro:property name="chassis_width" value="0.45" />
     <xacro:property name="chassis_height" value="0.25" />
-    <xacro:property name="chassis_mass" value="25.0" />
+    <xacro:property name="chassis_mass" value="5.0" />
     <xacro:property name="wheel_radius" value="0.1" />
     <xacro:property name="wheel_thickness" value="0.06" />
-    <xacro:property name="wheel_mass" value="1.5" />
+    <xacro:property name="wheel_mass" value="0.25" />
     <!-- Distance between left/right wheel centers and front/rear wheel centers -->
     <xacro:property name="track_width" value="0.5" />
