Commit message: update

File: src/urdfs/urdf/gazebo_plugin.xacro (robot description, xacro)
@@ -14,5 +14,5 @@
             <wheel_radius>0.05</wheel_radius>
             <frame_id>odom</frame_id>
-            <child_frame_id>roomba</child_frame_id>
+            <child_frame_id>zippy</child_frame_id>
         </plugin>
     </gazebo>

File: src/urdfs/urdf/ros2_hardwareinterface.xacro (robot description, xacro)
@@ -1,4 +1,4 @@
 <?xml version="1.0"?>
-<robot name="roomba" xmlns:xacro="https://www.ros.org/wiki/xacro">
+<robot name="zippy" xmlns:xacro="https://www.ros.org/wiki/xacro">
     <ros2_control name="GazeboSystem" type="system">
         <hardware>

File: src/urdfs/urdf/zippy.urdf.xacro (robot description, xacro)
@@ -1,4 +1,4 @@
 <?xml version="1.0"?>
-<robot name="roomba" xmlns:xacro="https://www.ros.org/wiki/xacro">
+<robot name="zippy" xmlns:xacro="https://www.ros.org/wiki/xacro">
     <xacro:arg name="controllers_config_path" default="" />
     <xacro:include filename="materials.xacro" />
@@ -9,14 +9,14 @@
     <xacro:include filename="gazebo_plugin.xacro" />
     <xacro:include filename="ros2_hardwareinterface.xacro" />
-    <xacro:property name="roomba_radius" value="0.2" />
-    <xacro:property name="roomba_height" value="0.1" />
+    <xacro:property name="zippy_radius" value="0.2" />
+    <xacro:property name="zippy_height" value="0.1" />
     <xacro:property name="wheel_radius" value="0.05" />
     <xacro:property name="wheel_thickness" value="0.03" />
-    <link name="roomba">
+    <link name="zippy">
     </link>
     <link name="base_link">
         <visual>
             <geometry>
-                <cylinder radius="${roomba_radius}" length="${roomba_height}" />
+                <cylinder radius="${zippy_radius}" length="${zippy_height}" />
             </geometry>
             <origin xyz="0 0 ${wheel_radius}" rpy="0 0 0" />
@@ -25,9 +25,9 @@
         <collision>
             <geometry>
-                <cylinder radius="${roomba_radius}" length="${roomba_height}" />
+                <cylinder radius="${zippy_radius}" length="${zippy_height}" />
             </geometry>
             <origin xyz="0 0 ${wheel_radius}" rpy="0 0 0" />
         </collision>
-        <xacro:cylinder_inertia Mass="10.0" r="${roomba_radius}" h="${roomba_height}" arr_xyz="0 0 ${wheel_radius}" arr_rpy="0 0 0" />
+        <xacro:cylinder_inertia Mass="10.0" r="${zippy_radius}" h="${zippy_height}" arr_xyz="0 0 ${wheel_radius}" arr_rpy="0 0 0" />
     </link>
     <xacro:macro name="wheel" params="params">
@@ -70,5 +70,5 @@
         <parent link="base_link"/>
         <child link="right_wheel"/>
-        <origin xyz="${-roomba_radius/2} ${-roomba_radius/2 - wheel_thickness/2} 0" rpy="0 0 0"/>
+        <origin xyz="${-zippy_radius/2} ${-zippy_radius/2 - wheel_thickness/2} 0" rpy="0 0 0"/>
         <axis xyz="0 1 0"/>
     </joint>
@@ -76,5 +76,5 @@
         <parent link="base_link"/>
         <child link="left_wheel"/>
-        <origin xyz="${-roomba_radius/2} ${roomba_radius/2 + wheel_thickness/2} 0" rpy="0 0 0"/>
+        <origin xyz="${-zippy_radius/2} ${zippy_radius/2 + wheel_thickness/2} 0" rpy="0 0 0"/>
         <axis xyz="0 1 0"/>
     </joint>
@@ -82,8 +82,8 @@
         <parent link="base_link"/>
         <child link="caster_wheel"/>
-        <origin xyz="${roomba_radius/4} 0 ${-wheel_radius/2}" rpy="0 0 0"/>
+        <origin xyz="${zippy_radius/4} 0 ${-wheel_radius/2}" rpy="0 0 0"/>
     </joint>
     <joint name="spine" type="fixed">
-        <parent link="roomba"/>
+        <parent link="zippy"/>
         <child link="base_link"/>
         <origin xyz="0 0 ${wheel_radius}" rpy="0 0 0"/>

Commit message: update

File: src/urdfs/urdf/gazebo_plugin.xacro (robot description, xacro)
@@ -9,5 +9,5 @@
             <right_joint>base_frontright_wheel_joint</right_joint>
             <right_joint>base_rearright_wheel_joint</right_joint>
-            <wheel_separation>0.5</wheel_separation>
+            <wheel_separation>0.51</wheel_separation>
             <wheel_radius>0.1</wheel_radius>
             <frame_id>odom</frame_id>

File: src/urdfs/urdf/zippy.urdf.xacro (robot description, xacro)
@@ -17,5 +17,5 @@
     <xacro:property name="wheel_mass" value="0.25" />
     <!-- Distance between left/right wheel centers and front/rear wheel centers -->
-    <xacro:property name="track_width" value="0.5" />
+    <xacro:property name="track_width" value="0.51" />
     <xacro:property name="wheelbase" value="0.45" />
     <!-- Height of the chassis center above the ground (wheel axle height) -->
